File: PCB/matrix.kicad_sch (KiCad schematic)
At the start: 27 parts, among them SW10 EC_SW, SW11 EC_SW, SW12 EC_SW, SW13 EC_SW, SW14 EC_SW, SW15 EC_SW, SW16 EC_SW, SW17 EC_SW, SW18 EC_SW, SW19 EC_SW, SW2 EC_SW, SW20 EC_SW, SW21 EC_SW, SW22 EC_SW, SW23 EC_SW, SW24 EC_SW, SW25 EC_SW, SW26 EC_SW, SW27 EC_SW, SW28 EC_SW, SW3 EC_SW, SW4 EC_SW, SW5 EC_SW, SW6 EC_SW, SW7 EC_SW, SW8 EC_SW, SW9 EC_SW

Commit message: Updated to `Rev 1.1`
Updated the title block in schematics to reflect company name and updated EC pads to latest model.
This update isn't critical, hence the lack of proper `Rev` update in README.
Other:
- company: Cipulot PCB Design -> LU.SV Solutions
- title: EC23U - Matrix -> EC23U
Changed lines of the file:
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@@
   (paper "A4")
   (title_block
-    (title "EC23U - Matrix")
-    (date "2022-11-18")
-    (rev "1")
-    (company "Cipulot PCB Design")
-    (comment 1 "MIT License")
-    (comment 2 "Cipulot")
+    (title "EC23U")
+    (date "2023-07-15")
+    (rev "1.1")
+    (company "LU.SV Solutions")
+    (comment 1 "Cipulot PCB Design")
+    (comment 2 "MIT License")
+    (comment 3 "Cipulot")
   )
   (junction (at 114.935 117.475) (diameter 0) (color 0 0 0 0)
