File: PCB/mounting_holes.kicad_sch (KiCad schematic)
At the start: 13 parts

Commit message: Updated to `Rev 1.1`
Updated the title block in schematics to reflect company name and updated EC pads to latest model.
This update isn't critical, hence the lack of proper `Rev` update in README.
Other:
- company: Cipulot PCB Design -> LU.SV Solutions
- title: EC23U - Mounting Holes -> EC23U
Changed lines of the file:
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@@
   (paper "A5")
   (title_block
-    (title "EC23U - Mounting Holes")
-    (date "2022-11-18")
-    (rev "1")
-    (company "Cipulot PCB Design")
-    (comment 1 "MIT License")
-    (comment 2 "Cipulot")
+    (title "EC23U")
+    (date "2023-07-15")
+    (rev "1.1")
+    (company "LU.SV Solutions")
+    (comment 1 "Cipulot PCB Design")
+    (comment 2 "MIT License")
+    (comment 3 "Cipulot")
   )
   (junction (at 63.5 67.31) (diameter 0) (color 0 0 0 0)
